Commit message: Add blank name to material

File: epick_description/urdf/helper_macros.xacro (robot description, xacro)
@@ -33,5 +33,5 @@
             <cylinder radius="${radius}" length="${length}"/>
           </geometry>
-          <material>
+          <material name="">
             <color rgba="${color}"/>
           </material>
