Commit message: Now using urdf in description package.

File: epick_description/urdf/epick_driver_ros2_control.xacro (robot description, xacro)
@@ -1,5 +1,5 @@
 <?xml version="1.0"?>
 <robot xmlns:xacro="http://www.ros.org/wiki/xacro">
-  <xacro:macro name="epick_ros2_control" params="name">
+  <xacro:macro name="epick_driver_ros2_control" params="name">
     <ros2_control name="${name}" type="system">
       <hardware>
@@ -7,5 +7,5 @@
        <!-- Serial connection parameters. -->
         <param name="usb_port">/dev/ttyUSB0</param>
-        <param name="baud_rate">9600</param>
+        <param name="baud_rate">115200</param>
         <param name="timeout">0.2</param>
         <!-- Gripper parameters. -->

File: epick_description/urdf/example.urdf.xacro (robot description, xacro)
@@ -1,7 +1,8 @@
 <?xml version="1.0"?>
-<robot xmlns:xacro="http://www.ros.org/wiki/xacro">
+<robot name="example_robot" xmlns:xacro="http://www.ros.org/wiki/xacro">
+  <xacro:include filename="$(find epick_description)/urdf/epick_single_suction_cup.xacro" ns="robotiq"/>
+  <xacro:include filename="$(find epick_description)/urdf/epick_driver_ros2_control.xacro" />
   <link name="world"/>
-  <!-- Attach EPick to world -->
-  <xacro:include filename="epick_single_suction_cup.xacro" ns="robotiq"/>
   <xacro:robotiq.epick_single_suction_cup parent="world"/>
+  <xacro:epick_driver_ros2_control name="epick_driver_ros2_control" />
 </robot>

Commit message: add ros2_control xacro to gripper description, add parameter for fake hardware

File: epick_description/urdf/epick_driver_ros2_control.xacro (robot description, xacro)
@@ -1,5 +1,5 @@
 <?xml version="1.0"?>
 <robot xmlns:xacro="http://www.ros.org/wiki/xacro">
-  <xacro:macro name="epick_driver_ros2_control" params="name">
+  <xacro:macro name="epick_driver_ros2_control" params="name use_fake_hardware:=true">
     <ros2_control name="${name}" type="system">
       <hardware>
@@ -11,5 +11,5 @@
         <!-- Gripper parameters /////////////////////////////////////////// -->
         <!-- Set use_dummy to true to connect to a dummy driver for testing purposes. -->
-        <param name="use_dummy">false</param>
+        <param name="use_dummy">${use_fake_hardware}</param>
         <!-- The address of the gripper. -->
         <param name="slave_address">0x9</param>

File: epick_description/urdf/epick_single_suction_cup.xacro (robot description, xacro)
@@ -3,4 +3,5 @@
   <!-- Include EPick Body and helper macros -->
   <xacro:include filename="epick_body.xacro"/>
+  <xacro:include filename="$(find epick_description)/urdf/epick_driver_ros2_control.xacro" />
   <!-- Robotiq EPick + Suction Cup with optional extension
        Creates the following kinematic chain of (prefixed) links:
@@ -30,4 +31,5 @@
                        extension_length:=0.0
                        tcp_stroke_compensation:=0.0">
+    <xacro:epick_driver_ros2_control name="epick_driver_ros2_control" />
     <!-- Body -->
     <!-- inherits prefix, parent and origin_*, exposes body_link, body_length, body_color -->

Commit message: add fake joint to represent vacuum state

File: epick_description/urdf/epick_driver_ros2_control.xacro (robot description, xacro)
@@ -11,5 +11,5 @@
         <!-- Gripper parameters /////////////////////////////////////////// -->
         <!-- Set use_dummy to true to connect to a dummy driver for testing purposes. -->
-        <param name="use_dummy">${use_fake_hardware}</param>
+        <param name="use_dummy">false</param>
         <!-- The address of the gripper. -->
         <param name="slave_address">0x9</param>

File: epick_description/urdf/epick_single_suction_cup.xacro (robot description, xacro)
@@ -67,4 +67,12 @@
                  child="${prefix}epick_tcp"
                  xyz="0 0 ${-tcp_stroke_compensation}"/>
+    <!-- To allow MoveIt to actuate the gripper as part of a trajectory, we need to include a fake "joint" in the URDF corresponding to the Epick's vacuum state. -->
+    <link name="${prefix}epick_vacuum_state"/>
+    <joint name="gripper" type="revolute">
+      <origin xyz="0 0 0" rpy="0 0 0"/>
+      <parent link="${prefix}epick_tcp"/>
+      <child link="${prefix}epick_vacuum_state"/>
+      <limit effort="30" velocity="1.0" lower="0.0" upper="1.0" />
+    </joint>
   </xacro:macro>
 </robot>

Commit message: Added "gripper/position" state interface.

File: epick_description/urdf/epick_driver_ros2_control.xacro (robot description, xacro)
@@ -30,5 +30,6 @@
         <command_interface name="grip_cmd"/>
         <!--
-          State interface that follow the value of the command interface:
+          State interface that follows the value of the gripper/grip_cmd
+          command interface:
           1.0 = successful grip
           0.0 = successful release
@@ -44,4 +45,17 @@
         <state_interface name="object_detection_status"/>
       </gpio>
+      <!--
+        This is optional configuration if you want to publish the state of the
+        gripper as a joint state interface.
+      -->
+      <joint name="gripper">
+        <!--
+          State interface that follows the value of the gripper/grip_cmd
+          command interface:
+          1.0 = successful grip
+          0.0 = successful release
+        -->
+        <state_interface name="position"/>
+      </joint>
     </ros2_control>
   </xacro:macro>

Commit message: Add parameters to the EPick ros2_control xacro file

File: epick_description/urdf/epick_driver_ros2_control.xacro (robot description, xacro)
@@ -1,24 +1,34 @@
 <?xml version="1.0"?>
 <robot xmlns:xacro="http://www.ros.org/wiki/xacro">
-  <xacro:macro name="epick_driver_ros2_control" params="name use_fake_hardware:=true">
+  <xacro:macro name="epick_driver_ros2_control"
+               params="name use_fake_hardware:=true
+                       usb_port:=/dev/ttyUSB0
+                       baud_rate:=115200
+                       timeout:=0.2
+                       slave_address:=0x9
+                       mode:=AdvancedMode
+                       grip_max_vacuum_pressure:=-60
+                       grip_min_vacuum_pressure:=-10
+                       grip_timeout:=25.0
+                       release_timeout:=2.0">
     <ros2_control name="${name}" type="system">
       <hardware>
         <plugin>epick_driver/EpickGripperHardwareInterface</plugin>
        <!-- Serial connection parameters ////////////////////////////////// -->
-        <param name="usb_port">/dev/ttyUSB0</param>
-        <param name="baud_rate">115200</param>
-        <param name="timeout">0.2</param>
+        <param name="usb_port">${usb_port}</param>
+        <param name="baud_rate">${baud_rate}</param>
+        <param name="timeout">${timeout}</param>
         <!-- Gripper parameters /////////////////////////////////////////// -->
         <!-- Set use_dummy to true to connect to a dummy driver for testing purposes. -->
         <param name="use_dummy">${use_fake_hardware}</param>
         <!-- The address of the gripper. -->
-        <param name="slave_address">0x9</param>
+        <param name="slave_address">${slave_address}</param>
         <!-- The gripper operation mode: AutomaticMode or AdvancedMode. -->
-        <param name="mode">AdvancedMode</param>
+        <param name="mode">${mode}</param>
         <!-- The following parameters are only required for the AdvancedMode. -->
-        <param name="grip_max_vacuum_pressure">-60</param>
-        <param name="grip_min_vacuum_pressure">-10</param>
-        <param name="grip_timeout">25.0</param>
-        <param name="release_timeout">2.0</param>
+        <param name="grip_max_vacuum_pressure">${grip_max_vacuum_pressure}</param>
+        <param name="grip_min_vacuum_pressure">${grip_min_vacuum_pressure}</param>
+        <param name="grip_timeout">${grip_timeout}</param>
+        <param name="release_timeout">${release_timeout}</param>
       </hardware>
       <gpio name="gripper">

File: epick_description/urdf/epick_single_suction_cup.xacro (robot description, xacro)
@@ -31,8 +31,11 @@
                        extension_length:=0.0
                        tcp_stroke_compensation:=0.0
-                       use_fake_hardware:=true">
+                       use_fake_hardware:=true
+                       usb_port:=/dev/ttyUSB0">
     <xacro:epick_driver_ros2_control
       name="epick_driver_ros2_control"
-      use_fake_hardware="${use_fake_hardware}"/>
+      use_fake_hardware="${use_fake_hardware}"
+      usb_port="${usb_port}"
+    />
     <!-- Body -->
     <!-- inherits prefix, parent and origin_*, exposes body_link, body_length, body_color -->

Commit message: Add action-based gripper controller (#7)
* Add GripperActionController-based Epick controller
* Move gripper status publishing to a separate controller
* Add epick_moveit_plugin package
* Add ros2_control xacro to gripper description, add parameter for fake hardware
* Add fake joint to represent vacuum state
* Add parameters to the EPick ros2_control xacro file (#21)

---------

Co-authored-by: marqrazz <marq.razz@gmail.com>
Co-authored-by: Sebastian Castro <sebas.a.castro@gmail.com>

File: epick_description/urdf/epick_driver_ros2_control.xacro (robot description, xacro)
@@ -1,24 +1,34 @@
 <?xml version="1.0"?>
 <robot xmlns:xacro="http://www.ros.org/wiki/xacro">
-  <xacro:macro name="epick_driver_ros2_control" params="name">
+  <xacro:macro name="epick_driver_ros2_control"
+               params="name use_fake_hardware:=true
+                       usb_port:=/dev/ttyUSB0
+                       baud_rate:=115200
+                       timeout:=0.2
+                       slave_address:=0x9
+                       mode:=AdvancedMode
+                       grip_max_vacuum_pressure:=-60
+                       grip_min_vacuum_pressure:=-10
+                       grip_timeout:=25.0
+                       release_timeout:=2.0">
     <ros2_control name="${name}" type="system">
       <hardware>
         <plugin>epick_driver/EpickGripperHardwareInterface</plugin>
        <!-- Serial connection parameters ////////////////////////////////// -->
-        <param name="usb_port">/dev/ttyUSB0</param>
-        <param name="baud_rate">115200</param>
-        <param name="timeout">0.2</param>
+        <param name="usb_port">${usb_port}</param>
+        <param name="baud_rate">${baud_rate}</param>
+        <param name="timeout">${timeout}</param>
         <!-- Gripper parameters /////////////////////////////////////////// -->
         <!-- Set use_dummy to true to connect to a dummy driver for testing purposes. -->
-        <param name="use_dummy">false</param>
+        <param name="use_dummy">${use_fake_hardware}</param>
         <!-- The address of the gripper. -->
-        <param name="slave_address">0x9</param>
+        <param name="slave_address">${slave_address}</param>
         <!-- The gripper operation mode: AutomaticMode or AdvancedMode. -->
-        <param name="mode">AdvancedMode</param>
+        <param name="mode">${mode}</param>
         <!-- The following parameters are only required for the AdvancedMode. -->
-        <param name="grip_max_vacuum_pressure">-60</param>
-        <param name="grip_min_vacuum_pressure">-10</param>
-        <param name="grip_timeout">25.0</param>
-        <param name="release_timeout">2.0</param>
+        <param name="grip_max_vacuum_pressure">${grip_max_vacuum_pressure}</param>
+        <param name="grip_min_vacuum_pressure">${grip_min_vacuum_pressure}</param>
+        <param name="grip_timeout">${grip_timeout}</param>
+        <param name="release_timeout">${release_timeout}</param>
       </hardware>
       <gpio name="gripper">

File: epick_description/urdf/epick_single_suction_cup.xacro (robot description, xacro)
@@ -3,4 +3,5 @@
   <!-- Include EPick Body and helper macros -->
   <xacro:include filename="epick_body.xacro"/>
+  <xacro:include filename="$(find epick_description)/urdf/epick_driver_ros2_control.xacro" />
   <!-- Robotiq EPick + Suction Cup with optional extension
        Creates the following kinematic chain of (prefixed) links:
@@ -29,5 +30,12 @@
                        extension_radius:=0.0
                        extension_length:=0.0
-                       tcp_stroke_compensation:=0.0">
+                       tcp_stroke_compensation:=0.0
+                       use_fake_hardware:=true
+                       usb_port:=/dev/ttyUSB0">
+    <xacro:epick_driver_ros2_control
+      name="epick_driver_ros2_control"
+      use_fake_hardware="${use_fake_hardware}"
+      usb_port="${usb_port}"
+    />
     <!-- Body -->
     <!-- inherits prefix, parent and origin_*, exposes body_link, body_length, body_color -->
@@ -65,4 +73,12 @@
                  child="${prefix}epick_tcp"
                  xyz="0 0 ${-tcp_stroke_compensation}"/>
+    <!-- To allow MoveIt to actuate the gripper as part of a trajectory, we need to include a fake "joint" in the URDF corresponding to the Epick's vacuum state. -->
+    <link name="${prefix}epick_vacuum_state"/>
+    <joint name="gripper" type="revolute">
+      <origin xyz="0 0 0" rpy="0 0 0"/>
+      <parent link="${prefix}epick_tcp"/>
+      <child link="${prefix}epick_vacuum_state"/>
+      <limit effort="30" velocity="1.0" lower="0.0" upper="1.0" />
+    </joint>
   </xacro:macro>
 </robot>
