Commit message: feat(description): make the gripper joint-state block opt-out
The macro unconditionally emits a <joint name="gripper"> state interface, guarded only by
a comment calling it optional. That element names a URDF joint, and ros2_control 4.x
validates every <ros2_control> joint against the assembled URDF: a name with no matching
joint makes parse_control_resources_from_urdf() throw, aborting ros2_control_node at
startup with SIGABRT.

Robots whose URDF has no joint literally called "gripper" therefore cannot use this macro
at all on Jazzy. A single-suction-cup EPick is exactly that case -- the cup is a chain of
fixed joints with no "gripper" among them -- so the reference is dangling and always was.
Humble simply never checked.

Adds publish_gripper_joint_state, defaulting to true so existing users on a robot that
does have such a joint see no change, and wraps the block in a xacro:if.

Co-Authored-By: Claude Opus 5 (1M context) <noreply@anthropic.com>

File: epick_description/urdf/epick_driver_ros2_control.xacro (robot description, xacro)
@@ -11,5 +11,6 @@
                        grip_min_vacuum_pressure:=-10
                        grip_timeout:=25.0
-                       release_timeout:=2.0">
+                       release_timeout:=2.0
+                       publish_gripper_joint_state:=true">
     <ros2_control name="${name}" type="system">
       <hardware>
@@ -58,14 +59,22 @@
         This is optional configuration if you want to publish the state of the
         gripper as a joint state interface.
+        It names a URDF joint, and ros2_control 4.x validates every
+        ros2_control joint against the URDF. A name with no matching joint
+        makes parse_control_resources_from_urdf() throw, which aborts
+        ros2_control_node at startup. Robots whose URDF has no joint literally
+        called "gripper" (a suction cup has none) must pass
+        publish_gripper_joint_state:=false.
       -->
-      <joint name="gripper">
-        <!--
-          State interface that follows the value of the gripper/grip_cmd
-          command interface:
-          1.0 = successful grip
-          0.0 = successful release
-        -->
-        <state_interface name="position"/>
-      </joint>
+      <xacro:if value="${publish_gripper_joint_state}">
+        <joint name="gripper">
+          <!--
+            State interface that follows the value of the gripper/grip_cmd
+            command interface:
+            1.0 = successful grip
+            0.0 = successful release
+          -->
+          <state_interface name="position"/>
+        </joint>
+      </xacro:if>
     </ros2_control>
   </xacro:macro>
